Commit message: impedant 3fgripper set up and tested

File: asset/robotiq_3f_gripper_visualization/cfg/robotiq-3f-gripper_articulated.urdf (robot description, URDF)
Before this commit: robot robotiq-3f-gripper_articulated, 13 links, 12 joints
Joints:
- joint finger_1_joint_1: limit lower=0 upper=3.1416 effort=100 velocity=100 -> lower=0 upper=3.1416 effort=1000 velocity=100
- joint finger_1_joint_2: limit lower=0 upper=3.1416 effort=100 velocity=100 -> lower=0 upper=3.1416 effort=1000 velocity=100
- joint finger_1_joint_3: limit lower=0 upper=3.1416 effort=100 velocity=100 -> lower=0 upper=3.1416 effort=1000 velocity=100
- joint finger_2_joint_1: limit lower=0 upper=3.1416 effort=100 velocity=100 -> lower=0 upper=3.1416 effort=1000 velocity=100
- joint finger_2_joint_2: limit lower=0 upper=3.1416 effort=100 velocity=100 -> lower=0 upper=3.1416 effort=1000 velocity=100
- joint finger_2_joint_3: limit lower=0 upper=3.1416 effort=100 velocity=100 -> lower=0 upper=3.1416 effort=1000 velocity=100
- joint finger_middle_joint_1: limit lower=0 upper=3.1416 effort=100 velocity=100 -> lower=0 upper=3.1416 effort=1000 velocity=100
- joint finger_middle_joint_2: limit lower=0 upper=3.1416 effort=100 velocity=100 -> lower=0 upper=3.1416 effort=1000 velocity=100
- joint finger_middle_joint_3: limit lower=0 upper=3.1416 effort=100 velocity=100 -> lower=0 upper=3.1416 effort=1000 velocity=100
- joint palm_finger_1_joint: limit lower=-0.16 upper=0.25 effort=100 velocity=100 -> lower=-0.16 upper=0.25 effort=1000 velocity=100
- joint palm_finger_2_joint: limit lower=-0.25 upper=0.16 effort=100 velocity=100 -> lower=-0.25 upper=0.16 effort=1000 velocity=100
- joint palm_finger_middle_joint: limit lower=-0.16 upper=0.25 effort=100 velocity=100 -> lower=-0.16 upper=0.25 effort=1000 velocity=100

Commit message: gripper implemented but vis incontinuity

File: asset/robotiq_3f_gripper_visualization/cfg/robotiq-3f-gripper_articulated.urdf (robot description, URDF)
Before this commit: robot robotiq-3f-gripper_articulated, 13 links, 12 joints
Joints:
- joint finger_1_joint_1: limit lower=0 upper=3.1416 effort=1000 velocity=100 -> lower=0 upper=0.65 effort=1000 velocity=0.1
- joint finger_1_joint_2: limit lower=0 upper=3.1416 effort=1000 velocity=100 -> lower=0 upper=0.65 effort=1000 velocity=0.1
- joint finger_1_joint_3: limit lower=0 upper=3.1416 effort=1000 velocity=100 -> lower=0 upper=0.65 effort=1000 velocity=0.1
- joint finger_2_joint_1: limit lower=0 upper=3.1416 effort=1000 velocity=100 -> lower=0 upper=0.65 effort=1000 velocity=0.1
- joint finger_2_joint_2: limit lower=0 upper=3.1416 effort=1000 velocity=100 -> lower=0 upper=0.65 effort=1000 velocity=0.1
- joint finger_2_joint_3: limit lower=0 upper=3.1416 effort=1000 velocity=100 -> lower=0 upper=0.65 effort=1000 velocity=0.1
- joint finger_middle_joint_1: limit lower=0 upper=3.1416 effort=1000 velocity=100 -> lower=0 upper=0.65 effort=1000 velocity=0.1
- joint finger_middle_joint_2: limit lower=0 upper=3.1416 effort=1000 velocity=100 -> lower=0 upper=0.65 effort=1000 velocity=0.1
- joint finger_middle_joint_3: limit lower=0 upper=3.1416 effort=1000 velocity=100 -> lower=0 upper=0.65 effort=1000 velocity=0.1
- joint palm_finger_1_joint: limit lower=-0.16 upper=0.25 effort=1000 velocity=100 -> lower=-0.16 upper=0.25 effort=1000 velocity=0.1
- joint palm_finger_2_joint: limit lower=-0.25 upper=0.16 effort=1000 velocity=100 -> lower=-0.25 upper=0.16 effort=1000 velocity=0.1
- joint palm_finger_middle_joint: limit lower=-0.16 upper=0.25 effort=1000 velocity=100 -> lower=-0.16 upper=0.25 effort=1000 velocity=0.1
