Commit message: shuffling test env done

File: asset/linkage.urdf (robot description, URDF)
Before this commit: robot linear_block_robot, 5 links, 4 joints
Links:
- link block1: geometry collision box size=1 0.35 3; visual box size=1 0.35 3
- link block2: geometry collision box size=1 0.35 3; visual box size=1 0.35 3
- link block3: geometry collision box size=1 0.35 3; visual box size=1 0.35 3
- link block4: geometry collision box size=1 0.35 3; visual box size=1 0.35 3
- link block5: geometry collision box size=1 0.35 3; visual box size=1 0.35 3

Commit message: shuffling example finished and tested; slow to find solutions - bad goal region?

File: asset/linkage.urdf (robot description, URDF)
Before this commit: robot linear_block_robot, 5 links, 4 joints
Joints:
- joint joint1: limit lower=-1.57 upper=1.57 effort=1000 velocity=50 -> lower=-.57 upper=.57 effort=1000 velocity=50
- joint joint2: limit lower=-1.57 upper=1.57 effort=1000 velocity=50 -> lower=-.57 upper=.57 effort=1000 velocity=50
- joint joint3: limit lower=-1.57 upper=1.57 effort=1000 velocity=50 -> lower=-.57 upper=.57 effort=1000 velocity=50
- joint joint4: limit lower=-1.57 upper=1.57 effort=1000 velocity=50 -> lower=-.57 upper=.57 effort=1000 velocity=50
