Commit message: obj urdf added

File: asset/real-world/concave-object/concave-object.urdf (robot description, URDF)
Before this commit: robot circle-gripper, 1 links, 0 joints
Links:
- link base_link: mass 26 -> 43; geometry collision mesh filename=package://asset/real-world/concave-object/concave-object-vh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 scale=1 1 1; visual mesh filename=package://asset/real-world/concave-object/concave-object-vh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 scale=1 1 1

File: asset/real-world/convex-object/convex-object.urdf (robot description, URDF)
Before this commit: robot circle-gripper, 1 links, 0 joints
Links:
- link base_link: mass 26 -> 42; geometry collision mesh filename=package://asset/real-world/convex-object/convex-object.obj scale=1 1 1; visual mesh filename=package://asset/real-world/convex-object/convex-object.obj scale=1 1 1

File: asset/real-world/irregular-object/irregular-object.urdf (robot description, URDF)
Before this commit: robot irregular-object, 1 links, 0 joints
Links:
- link base_link: mass 10 -> 24

File: asset/real-world/jaw-gripper/jaw-gripper.urdf (robot description, URDF)
Before this commit: robot circle-gripper, 1 links, 0 joints
Links:
- link base_link: geometry collision mesh filename=package://asset/real-world/jaw-gripper/jaw-gripper-vhacd.obj scale=1 1 1; visual mesh filename=package://asset/real-world/jaw-gripper/jaw-gripper-vhacd.obj scale=1 1 1

File: asset/real-world/rectangle-object/rectangle-object.urdf (robot description, URDF)
Before this commit: robot rectangle-object, 1 links, 0 joints
Links:
- link base_link: mass 10 -> 49

File: asset/real-world/triangle-object/triangle-object.urdf (robot description, URDF)
Before this commit: robot circle-gripper, 1 links, 0 joints
Links:
- link base_link: mass 26 -> 28; geometry collision mesh filename=package://asset/real-world/triangle-object/triangle-object.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 scale=1 1 1; visual mesh filename=package://asset/real-world/triangle-object/triangle-object.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 scale=1 1 1
