Commit message: gripper multi ellipse dataset half-run

File: asset/lc_soft_enable_wide_grip/lc_soft_enable_wide_grip.urdf (robot description, URDF)
Before this commit: robot lc_soft_enable_wide_grip, 5 links, 4 joints
Joints:
- joint left_base: origin xyz=0.07658 4.689172593935216e-18 0.1335 rpy=1.874699728327322e-33 -1.5707963057214722 0 -> xyz=0.06658 4.689172593935216e-18 0.1335 rpy=1.874699728327322e-33 -1.5707963057214722 0
- joint right_finger: origin xyz=-0.07658 -4.689172593935216e-18 0.1335 rpy=-3.141592653589793 -1.5707963057214722 0 -> xyz=-0.06658 -4.689172593935216e-18 0.1335 rpy=-3.141592653589793 -1.5707963057214722 0
